File: PCB/DiabloController.sch (KiCad schematic (older format))
At the start: 44 parts, among them J1 CONN_02X25, U1 74LVC04, U2 74LS04, U3 74LS04, U4 74LS04, U5 74LSV04, U6 74LSV04, U7 STM32BluePill

Commit message: Updated schematic for the patches done
Parts:
- added R19, R20, R21, R22, R23, R24, R25, R26, R27, R28, R29, R30, R31, R32, R33, R34, R35, R36, R37: R, Resistors_SMD:R_0805_HandSoldering, symbol R
Connections:
- net GND: now also R19.2, R20.2, R21.2, R22.2, R23.2, R24.2, R25.2, R26.2, R27.2, R28.2, R29.2, R30.2, R31.2, R32.2, R33.2, R34.2, R35.2, R36.2, R37.1
- net PCarStr: now also R33.1
- net PDB1: now also R19.1
- net PDB10: now also U7.22 (PC13), R28.1; no longer U7.6 (PA9)
- net PDB11: now also U7.23 (PC14), R29.1; no longer U7.7 (PA10)
- net PDB12: now also U7.24 (PC15), R30.1; no longer U7.8 (PA11)
- net PDB2: now also R20.1
- net PDB3: now also R21.1
- net PDB4: now also R22.1
- net PDB5: now also R23.1
- net PDB6: now also R24.1
- net PDB7: now also R25.1
- net PDB8: now also R26.1
- net PDB9: now also R27.1
- net POptStr: now also R34.1
- net PPFStr: now also R32.1
- net PPWStr: now also R35.1
- net PRestore: now also R31.1
- net PRibLift: now also R36.1
- net PSelPrt: now also R37.2

Commit message: Some components got lost in the move. Fixed automatically by KiCad
Parts:
- C1, C2, C3, C4, C5, C6, C7, C8, C9: symbol C -> DiabloController-rescue:C
- D1, D16, D2, D3, D4, D5, D6, D7, D8: symbol LED -> DiabloController-rescue:LED
- J1: symbol CONN_02X25 -> DiabloController-rescue:CONN_02X25
- R1, R10, R11, R12, R13, R14, R15, R16, R17, R18, R19, R2, R20, R21, R22, R23, R24, R25, R26, R27, R28, R29, R3, R30, R31, R32, R33, R34, R35, R36, R37, R4, R5, R6, R7, R8, R9: symbol R -> DiabloController-rescue:R
- U1, U2, U3, U4: symbol 74LS04 -> DiabloController-rescue:74LS04
- U5, U6: symbol 74LSV04 -> DiabloController-rescue:74LSV04
- U7: symbol STM32BluePill-RESCUE-DiabloController -> DiabloController-rescue:STM32BluePill-RESCUE-DiabloController
